Commit message: fix(assets): zero motor joint_vel + prop inertials + Sim 5.1 mass patch
Sim 5.1 ContactSensor returns phantom 76-1869 N on the drone body at rest.
Two root causes addressed here:

- Props had no <inertial> in URDF, so Isaac Sim assigned defaults that overshot
  total drone mass ~1000x. Add <inertial> (m=0.025 kg, diag I=(1e-6, 1e-6, 2e-6))
  to prop1..prop4 and patch the live USD files via scripts/patch_drone_usd_mass.py
  (sets body to 0.5 kg with diag inertia (0.003, 0.003, 0.006)).
- joint_vel init was {m1:200, m2:-200, m3:200, m4:-200}. Spinning props at reset
  generated bogus gyroscopic torques and feed into the propeller spin-up that
  exaggerates phantom contact transients. Replace with {".*": 0.0}.

Co-Authored-By: Claude Opus 4.7 <noreply@anthropic.com>

File: assets/5_in_drone/urdf/5_in_drone.urdf (robot description, URDF)
Before this commit: robot 5_in_drone, 5 links, 4 joints
Links:
- link prop1: mass None -> 0.025
- link prop2: mass None -> 0.025
- link prop3: mass None -> 0.025
- link prop4: mass None -> 0.025
